File: hard/ekdome/ekdome.kicad_sch (KiCad schematic)
At the start: 92 parts, among them J10 USB_P, J11 DBG, J20 HBS, J21 HBS, J22 HPW, J30 POWER, Q20 SS8050, Q21 SS8050, U10 CH32V203C8T6, U11 CH340E, U13 74LVC1G86, U20 MS1192, U30 XL1509, U31 AMS1117-3.3, Y10 12M

Commit message: V1.1 complete
Parts:
- removed J22: HPW, kicad_footprint_general:PhoenixContact_MCV_1,5_2-G-3.81_1x02_P3.81mm_Vertical, symbol kicad_symbol_general:Conn_01x02
- removed L20, L21: 100mH, symbol kicad_symbol_general_s:L_Small
- added C101: 100nF, kicad_footpring_general:C_0603_1608Metric, symbol kicad_symbol_general:C_Small
- added R18: 1k, kicad_footpring_general:R_0603_1608Metric, symbol kicad_symbol_general:R_Small_US
- added R204: 10k, kicad_footpring_general:R_0603_1608Metric, symbol kicad_symbol_general:R_Small_US
- added TL10, TL11, TL20, TL21: L, TestPoint:TestPoint_Loop_D2.50mm_Drill1.0mm, symbol Connector:TestPoint
- C201, C27: footprint kicad_footprint_general:C_0603_1608Metric -> kicad_footpring_general:C_0603_1608Metric
- Q20, Q21: value SS8050 -> NP
- R20: value 330R -> 220R
- R203: footprint kicad_footprint_general:R_0603_1608Metric -> kicad_footpring_general:R_0603_1608Metric
- R21: value 510R -> NP
- R27, R28: value 1.6R -> 1.0R; footprint kicad_footprint_general:R_0603_1608Metric -> kicad_footpring_general:R_0603_1608Metric
- U13: footprint kicad_footprint_general:SOT-23-5 -> kicad_footpring_general:SOT-23-5; symbol kicad_symbol_general:74LVC1G86 -> kicad_symbol_general_s:74LVC1G86
Connections:
- net +18V: now also D30.1 (K), D31.4, TL20.1; no longer C21.1, C23.1, J20.1 (Pin_1), J21.1 (Pin_1), R201.1
- net +5V: now also R204.1
- net CFT: now also C101.1, R18.2; no longer U13.4
- net GND: now also C101.2
- net at R20.1, U20.1 (DOUT): now also R204.2
- net at C22.1, C24.1, J20.2 (Pin_2)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: now also J21.1 (Pin_1), TL11.1; no longer J21.2 (Pin_2)
- net at D31.3, J30.1 (Pin_1): now also TL10.1
- new net: C21.1, C23.1, J20.1 (Pin_1), J21.2 (Pin_2), R201.1, TL21.1
- new net: R18.1, U13.4
Other:
- moved on the sheet: C100, U13
